File: hw/gun.sch (KiCad schematic (older format))
At the start: 46 parts, among them J1 SWD_01X04, J2 IDC_02X05, SW1 FUSE, SW2 BANG, U1 OSRB38C9BA, U2 ULN2003, U3 74AHC1G08, U4 MCP1826S, U5 STM32F042F6Px, U6 MCP1826S

Commit message: updated schematic
Parts:
- added C1, C6: 100n, symbol Device:C
- added R13, R14: 100R, symbol Device:R
- added U2: ULN2003, symbol Transistor_Array:ULN2003
- added U7, U9: 74AHC1G08, Package_TO_SOT_SMD:SOT-23-5, symbol KLIB_Logic:74AHC1G08
- D5, D6: footprint LEDs:LED_WS2812-PLCC6 -> KLIB_Opto:LED_RGB_5050-6
- J2: footprint Connectors:IDC_Header_Straight_10pins -> Connector_IDC:IDC-Header_2x05_P2.54mm_Vertical
- U1: footprint (none) -> KLIB_Opto:OSRB8C9BA_Vertical
- renumbered C5 to C10, C6 to C11, C7 to C12, C8 to C13, C10 to C14, C9 to C15, C11 to C16, C12 to C2, C13 to C3, C1 to C4, C14 to C5, C2 to C7, C3 to C8, C4 to C9, D3 to D1, D1 to D3, U2 to U3, U3 to U5, U5 to U6, U6 to U8
Connections:
- net +3V3: now also C1.1, C6.1
- net +5V: now also U7.5 (VCC), U9.5 (VCC)
- net +5V5: now also U2.9 (COM)
- net BANG: now also R14.1; no longer C16.1
- net FUSE: now also R13.1; no longer C15.1
- net GND: now also C1.2, C6.2, U2.8 (GND), U7.3 (GND), U9.3 (GND)
- net GUN_RX: now also U6.18 (I2C1_SDA/TIM17_BKIN/TIM1_CH3/TSC_G4_IO2/USART1_RX/CAN_TX/TIM1_ETR/TSC_G4_IO4/USB_DP/PA12/PA10), U9.4 (Y); no longer J2.5, J2.6, U6.9 (ADC_IN3/TIM2_CH4/TSC_G1_IO4/USART2_RX/PA3)
- net GUN_TX: now also U6.17 (I2C1_SCL/TIM1_CH2/TSC_G4_IO1/USART1_TX/CAN_RX/I2C1_SCL/TIM1_CH4/TSC_G4_IO3/USB_DM/PA11/PA9), U7.1 (A), U7.2 (B); no longer J2.7, J2.8, U6.8 (ADC_IN2/SYS_WKUP4/TIM2_CH3/TSC_G1_IO3/USART2_TX/PA2)
- net IR_TX: now also U6.8 (ADC_IN2/SYS_WKUP4/TIM2_CH3/TSC_G1_IO3/USART2_TX/PA2); no longer U6.17 (I2C1_SCL/TIM1_CH2/TSC_G4_IO1/USART1_TX/CAN_RX/I2C1_SCL/TIM1_CH4/TSC_G4_IO3/USB_DM/PA11/PA9)
- net LED_IR: now also U2.1 (I1), U2.2 (I2), U2.3 (I3), U2.4 (I4); no longer U3.3 (I3)
- net LED_UV: now also U2.5 (I5), U2.6 (I6), U2.7 (I7); no longer U3.2 (I2)
- net LED_WH: now also U3.2 (I2), U3.3 (I3)
- net at R5.2, U3.14 (O3): now also U3.15 (O2), U3.16 (O1)
- net at R3.2: now also U2.10 (O7), U2.11 (O6), U2.12 (O5); no longer U3.15 (O2)
- net at R2.2: now also U2.13 (O4), U2.14 (O3), U2.15 (O2), U2.16 (O1); no longer U3.16 (O1)
- net at D3.1 (K): now also R5.1; no longer R2.1
- net at D1.1 (K): now also R2.1; no longer R5.1
- new net: C15.1, R13.2
- new net: C16.1, R14.2
- new net GUN_UART_RX: J2.5, J2.6, U9.1 (A), U9.2 (B)
- new net GUN_UART_TX: J2.7, J2.8, U7.4 (Y)
Other:
- moved on the sheet: C10, C11, C12, C13, C14, C15, C16, C2, C3, C4, C5, C7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

Commit message: updated schematic
Parts:
- C1, C12, C13, C15, C16, C2, C3, C5, C6, C8, C9: footprint (none) -> Capacitor_SMD:C_0805_2012Metric
- C10, C11, C14, C7: value 1u -> 1u/50V; footprint (none) -> Capacitor_SMD:C_0805_2012Metric
- C4: footprint (none) -> Capacitor_Tantalum_SMD:CP_EIA-7343-31_Kemet-D
- D1, D2, D3, D4: footprint (none) -> Connector_PinHeader_2.54mm:PinHeader_1x02_P2.54mm_Vertical
- R1, R10, R11, R12, R13, R14, R4, R7, R8, R9: footprint (none) -> Resistor_SMD:R_0805_2012Metric
- R2, R3, R5, R6: footprint (none) -> Resistor_SMD:R_1210_3225Metric
- SW1, SW2: footprint (none) -> Connector_PinHeader_2.54mm:PinHeader_2x01_P2.54mm_Vertical
- U2, U3: footprint (none) -> Package_SO:SOIC-16_3.9x9.9mm_P1.27mm
Other:
- moved on the sheet: C10, C11, C12, C13, C14, C7, C8, C9, U4, U8

Commit message: updated schematic
Connections:
- net +3V3: no longer C5.1, C6.1
- net +5V: now also C5.1, C6.1
Changed lines of the file:
@@
 Wire Wire Line
 	1750 1000 1750 950
-Connection ~ 1750 950
-Wire Wire Line
-	1750 950  2200 950
 $Comp
 L KLIB_Power:GND #PWR05
 U 1 1 5ACB70B0
-P 1750 1400
-F 0 "#PWR05" H 1750 1200 50  0001 C CNN
-F 1 "GND" H 1755 1227 50  0000 C CNN
-F 2 "" H 1750 1400 50  0001 C CNN
-F 3 "" H 1750 1400 50  0001 C CNN
-	1    1750 1400
+P 1300 1400
+F 0 "#PWR05" H 1300 1200 50  0001 C CNN
+F 1 "GND" H 1305 1227 50  0000 C CNN
+F 2 "" H 1300 1400 50  0001 C CNN
+F 3 "" H 1300 1400 50  0001 C CNN
+	1    1300 1400
 	1    0    0    -1
 $EndComp
@@
 Wire Wire Line
 	2200 1350 2200 1300
-Wire Wire Line
-	1750 1400 1750 1350
-Connection ~ 1750 1350
-Wire Wire Line
-	1750 1350 2200 1350
 Wire Wire Line
 	1750 1300 1750 1350
@@
 L KLIB_Power:+3V3 #PWR04
 U 1 1 5ACC8036
-P 1750 900
-F 0 "#PWR04" H 1750 600 50  0001 C CNN
-F 1 "+3V3" H 1755 1073 50  0000 C CNN
-F 2 "" H 1750 900 50  0001 C CNN
-F 3 "" H 1750 900 50  0001 C CNN
-	1    1750 900
-	1    0    0    -1
-$EndComp
-Wire Wire Line
-	1750 900  1750 950
+P 1300 900
+F 0 "#PWR04" H 1300 600 50  0001 C CNN
+F 1 "+3V3" H 1305 1073 50  0000 C CNN
+F 2 "" H 1300 900 50  0001 C CNN
+F 3 "" H 1300 900 50  0001 C CNN
+	1    1300 900
+	1    0    0    -1
+$EndComp
 $Comp
 L KLIB_Mechanical:Bolt H1
@@
 Connection ~ 1300 950
 Wire Wire Line
-	2200 950  2650 950
+	2200 950  2450 950
 Wire Wire Line
 	2650 950  2650 1000
-Connection ~ 2200 950
 Wire Wire Line
 	2650 1300 2650 1350
 Wire Wire Line
-	2650 1350 2200 1350
-Connection ~ 2200 1350
+	2650 1350 2450 1350
 Wire Wire Line
 	1300 1350 850  1350
@@
 Wire Wire Line
 	3450 900  3450 950
+Wire Wire Line
+	1300 900  1300 950
+Wire Wire Line
+	1300 1400 1300 1350
+$Comp
+L KLIB_Power:+5V #PWR?
+U 1 1 5B5EC82F
+P 2450 900
+F 0 "#PWR?" H 2450 600 50  0001 C CNN
+F 1 "+5V" H 2455 1073 50  0000 C CNN
+F 2 "" H 2450 900 50  0001 C CNN
+F 3 "" H 2450 900 50  0001 C CNN
+	1    2450 900
+	1    0    0    -1
+$EndComp
+$Comp
+L KLIB_Power:GND #PWR?
+U 1 1 5B5EC8AB
+P 2450 1400
+F 0 "#PWR?" H 2450 1200 50  0001 C CNN
+F 1 "GND" H 2455 1227 50  0000 C CNN
+F 2 "" H 2450 1400 50  0001 C CNN
+F 3 "" H 2450 1400 50  0001 C CNN
+	1    2450 1400
+	1    0    0    -1
+$EndComp
+Wire Wire Line
+	2450 1400 2450 1350
+Connection ~ 2450 1350
+Wire Wire Line
+	2450 1350 2200 1350
+Wire Wire Line
+	2450 900  2450 950
+Connection ~ 2450 950
+Wire Wire Line
+	2450 950  2650 950
 $EndSCHEMATC

Commit message: updated pcb
Connections:
- net +5V: now also U2.9 (COM), U3.9 (COM)
- net +5V5: no longer U2.9 (COM), U3.9 (COM)
- net LED_UV: now also U6.1 (PB8/CAN_RX/CEC/I2C1_SCL/TIM16_CH1/TSC_SYNC); no longer U6.2 (PF0/CRS_SYNC/I2C1_SDA/RCC_OSC_IN)
- net LED_WH: now also U6.2 (PF0/CRS_SYNC/I2C1_SDA/RCC_OSC_IN); no longer U6.1 (PB8/CAN_RX/CEC/I2C1_SCL/TIM16_CH1/TSC_SYNC)
Changed lines of the file:
@@
 	650  7300 1050 7300
-$Comp
-L KLIB_Power:+5V5 #PWR08
-U 1 1 5AC01DF6
-P 1950 6450
-F 0 "#PWR08" H 1950 6150 50  0001 C CNN
-F 1 "+5V5" H 1955 6623 50  0000 C CNN
-F 2 "" H 1950 6450 50  0001 C CNN
-F 3 "" H 1950 6450 50  0001 C CNN
-	1    1950 6450
-	1    0    0    -1
-$EndComp
 $Comp
 L Device:R R9
@@
 Wire Wire Line
 	3350 3150 2950 3150
-Text Label 2950 3150 0    50   ~ 0
+Text Label 2950 2750 0    50   ~ 0
 LED_WH
 Text Label 9550 2150 2    50   ~ 0
@@
 	9350 900  9850 900
 Connection ~ 9850 900
-Text Label 2950 2750 0    50   ~ 0
+Text Label 2950 3150 0    50   ~ 0
 LED_UV
 Wire Wire Line
@@
 Wire Wire Line
 	1000 5500 1000 5600
-$Comp
-L KLIB_Power:+5V5 #PWR09
-U 1 1 5B41BD2C
-P 1900 4750
-F 0 "#PWR09" H 1900 4450 50  0001 C CNN
-F 1 "+5V5" H 1905 4923 50  0000 C CNN
-F 2 "" H 1900 4750 50  0001 C CNN
-F 3 "" H 1900 4750 50  0001 C CNN
-	1    1900 4750
-	1    0    0    -1
-$EndComp
 Wire Wire Line
 	1850 4800 1900 4800
@@
 	1300 1400 1300 1350
 $Comp
-L KLIB_Power:+5V #PWR?
+L KLIB_Power:+5V #PWR0101
 U 1 1 5B5EC82F
 P 2450 900
-F 0 "#PWR?" H 2450 600 50  0001 C CNN
+F 0 "#PWR0101" H 2450 600 50  0001 C CNN
 F 1 "+5V" H 2455 1073 50  0000 C CNN
 F 2 "" H 2450 900 50  0001 C CNN
@@
 $EndComp
 $Comp
-L KLIB_Power:GND #PWR?
+L KLIB_Power:GND #PWR0102
 U 1 1 5B5EC8AB
 P 2450 1400
-F 0 "#PWR?" H 2450 1200 50  0001 C CNN
+F 0 "#PWR0102" H 2450 1200 50  0001 C CNN
 F 1 "GND" H 2455 1227 50  0000 C CNN
 F 2 "" H 2450 1400 50  0001 C CNN
@@
 Wire Wire Line
 	2450 950  2650 950
+$Comp
+L KLIB_Power:+5V #PWR0103
+U 1 1 5B60711F
+P 1900 4750
+F 0 "#PWR0103" H 1900 4450 50  0001 C CNN
+F 1 "+5V" H 1905 4923 50  0000 C CNN
+F 2 "" H 1900 4750 50  0001 C CNN
+F 3 "" H 1900 4750 50  0001 C CNN
+	1    1900 4750
+	1    0    0    -1
+$EndComp
+$Comp
+L KLIB_Power:+5V #PWR0104
+U 1 1 5B607194
+P 1950 6450
+F 0 "#PWR0104" H 1950 6150 50  0001 C CNN
+F 1 "+5V" H 1955 6623 50  0000 C CNN
+F 2 "" H 1950 6450 50  0001 C CNN
+F 3 "" H 1950 6450 50  0001 C CNN
+	1    1950 6450
+	1    0    0    -1
+$EndComp
 $EndSCHEMATC
