File: hw/gun.kicad_pcb (KiCad board)
At the start: 2 copper layers, 65 x 45 mm, 53 parts, among them J1 SWD_01X04, J2 IDC_02X05, SW1 FUSE, SW2 BANG, U1 OSRB38C9BA, U2 ULN2003, U3 ULN2003, U4 MCP1826S, U5 74AHC1G08, U6 STM32F042F6Px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

Commit message: updated pcb
Parts:
- moved R10 39.8 mm to (178.5, 122.0)
- moved R11 35.8 mm to (178.5, 120.0)
- moved R12 32.0 mm to (178.5, 118.0)
- moved D6 19.1 mm to (162.5, 97.5), turned to 270 degrees
- moved D5 16.3 mm to (162.5, 112.5), turned to 90 degrees
- moved C11 14.3 mm to (164.8, 90.8)
- moved C12 14.3 mm to (166.8, 90.8)
- moved C13 14.3 mm to (176.2, 90.8)
- moved C14 14.3 mm to (178.2, 90.8)
- moved U8 14.3 mm to (171.5, 90.8)
- moved R7 10.3 mm to (160.5, 119.0), turned to 270 degrees
- moved R1 9.36 mm to (142.5, 112.8), turned to 0 degrees
- moved R8 8.31 mm to (162.5, 119.0), turned to 270 degrees
- moved U3 7.25 mm to (171.5, 115.5)
- moved R9 6.93 mm to (164.5, 119.0), turned to 270 degrees
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Other:
- board size 65 x 45 mm -> 65 x 40 mm

Commit message: updated pcb
Routing:
- net +5V: track 0.00 -> 108.6 mm, vias 0 -> 3
- net Net-(D6-Pad1): track 0.00 -> 36.8 mm, vias 0 -> 2
- net +5V5: track 0.00 -> 35.2 mm, vias 0 -> 3
- net Net-(D6-Pad2): track 0.00 -> 34.0 mm, vias 0 -> 2
- net Net-(D6-Pad3): track 0.00 -> 31.4 mm, vias 0 -> 2
- net /IR_RX: track 0.00 -> 21.2 mm
- net /GUN_UART_TX: track 0.00 -> 13.2 mm
- net /GUN_UART_RX: track 0.00 -> 12.7 mm
- net Net-(R2-Pad2): track 0.00 -> 9.47 mm
- net Net-(R5-Pad2): track 0.00 -> 7.67 mm
- net Net-(R3-Pad2): track 0.00 -> 6.97 mm
- net +3V3: track 0.00 -> 6.39 mm
- net Net-(R10-Pad2): track 0.00 -> 5.93 mm
- net Net-(R11-Pad2): track 0.00 -> 4.90 mm
- net Net-(R6-Pad2): track 0.00 -> 4.60 mm
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- added copper zone on B.Cu, net GND
- added copper zone on F.Cu, net GND

Commit message: updated pcb
Parts:
- moved C3 1.12 mm to (152.5, 111.0)
- moved U5 1.12 mm to (149.5, 111.0)
Connections:
- U2 pad 9: +5V5 -> +5V
- U3 pad 9: +5V5 -> +5V
- U6 pad 1: /LED_WH -> /LED_UV
- U6 pad 2: /LED_UV -> /LED_WH
Routing:
- net +3V3: track 6.39 -> 65.6 mm, vias 0 -> 5
- net +5V: track 108.6 -> 150.4 mm, vias 3 -> 9
- net /LED_WH: track 2.54 -> 38.2 mm, vias 0 -> 2
- net /BANG: track 2.87 -> 38.1 mm
- net /GUN_RX: track 0.00 -> 34.8 mm
- net /GUN_TX: track 0.00 -> 31.1 mm
- net /LASER: track 0.00 -> 30.1 mm, vias 0 -> 2
- net /LED_UV: track 2.54 -> 30.3 mm, vias 0 -> 2
- net /LED_IR: track 3.81 -> 30.8 mm, vias 0 -> 2
- net /PWM_B: track 0.00 -> 21.8 mm
- net /PWM_G: track 0.00 -> 21.2 mm
- net /FUSE: track 2.87 -> 23.8 mm
- net /PWM_R: track 0.00 -> 20.6 mm
- net Net-(R10-Pad2): track 5.93 -> 23.9 mm
- net Net-(R11-Pad2): track 4.90 -> 21.0 mm
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
Commit message: update pcb
Routing:
- net +5V: track 150.4 -> 199.0 mm, vias 9 -> 11
- net +3V3: track 65.6 -> 89.7 mm, vias 5 -> 6
- net GND: track 0.00 -> 4.66 mm, vias 0 -> 36
- net /LED_IR: track 30.8 -> 32.5 mm
- net /GUN_RX: track 34.8 -> 34.0 mm

Commit message: updated pcb
Routing:
- net /GUN_TX: track 30.7 -> 29.7 mm
- net /GUN_RX: track 34.0 -> 33.1 mm
- net /FUSE: track 23.8 -> 24.4 mm
- net GND: vias 36 -> 62

Commit message: updated pcb
Parts:
- added G***: LOGO, KLIB_Logo:wykys_small_skill, F.Cu at (156.0, 91.0)
- added REF**: Fiducial_Pad_1mm_Outer_2mm, KLIB_Mechanical:Fiducial_Pad_1mm_Outer_2mm, F.Cu at (181.0, 94.0)
- added REF**: Fiducial_Pad_1mm_Outer_2mm, KLIB_Mechanical:Fiducial_Pad_1mm_Outer_2mm, F.Cu at (130.0, 114.0)
- added REF**: Fiducial_Pad_1mm_Outer_2mm, KLIB_Mechanical:Fiducial_Pad_1mm_Outer_2mm, F.Cu at (130.0, 96.0)
Routing:
- net GND: vias 62 -> 54
Other:
- board text added: "GUN V3"
